File: kicad/Untitled.kicad_sch (KiCad schematic)
At the start: 10 parts, among them J1 2-171825-3, J2 2-171825-3, J3 2-171825-3, J4 2-171825-3, J5 171825-2, J6 171825-6, U1 esp32_38_pins-custom_library, U2 MPU-6050

Commit message: updated pcb
Parts:
- U2: footprint Sensor_Motion:InvenSense_QFN-24_4x4mm_P0.5mm -> GY-521:MODULE_GY-521
Changed lines of the file:
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@@
 			)
 		)
-		(property "Footprint" "Sensor_Motion:InvenSense_QFN-24_4x4mm_P0.5mm"
+		(property "Footprint" "GY-521:MODULE_GY-521"
 			(at 189.23 104.14 0)
 			(effects
